File: DX32G.kicad_pcb (KiCad board)
At the start: 2 copper layers, 53.3 x 45.7 mm, 35 parts, among them J1 USB_B_Micro, J2 MicroSD Card, J3 RIGHT, J4 LEFT, J7 USB_B_Micro, SW1 reset, SW2 boot, U1 ESP32-S3-WROOM-1, U2 AMS1117-3.3, U3 CH340N

Commit message: fixed minor silkscreen mistakes
Parts:
- removed TP3: IO_48, TestPoint:TestPoint_Pad_1.5x1.5mm
Routing:
- net /RGB_LED: track 26.5 -> 7.61 mm
- net /BOOT: track 35.0 -> 40.5 mm
Other:
- board text added: "4"
- board text added: "IO15"
- board text added: "Version 1.1"
- board text added: "WayWayWay"
- board text removed: "14"
- board text removed: "48"
